File: pcb/revA.kicad_pcb (KiCad board)
At the start: 2 copper layers, 68 x 49.3 mm, 45 parts, among them P1 USB_OTG, P2 EXP, P3 espprog, P4 BAT, P5 SAMD-PROG, P6 SPI-EXPANSION, SW1 SPST, U1 AP2112K-3.3, U2 SAMD20G18A-M, U3 MCP73831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

Commit message: Updated PCB to the version shipping to kickstarter backers :+1:
Parts:
- removed TyroBot: , components:tyrobot
- added tyrobotlogo: , components:tyrobotlogo, F.Cu at (111.9, 90.3)
- P3: footprint user:espprog -> Pin_Headers:Pin_Header_Straight_1x04_Pitch2.54mm
- moved P3 8.06 mm to (169.4, 79.1), turned to 0 degrees
Routing:
- net /ESP-GPIO0: track 6.46 -> 26.0 mm, vias 0 -> 1
- net /RXD: track 43.8 -> 55.5 mm
- net /TXD: track 41.0 -> 46.6 mm
- net /ESP-~RESET: track 28.2 -> 32.3 mm
Other:
- board text added: "P0"
- board text added: "REV A"
- board text added: "RST"
- board text added: "RX"
- board text added: "TX"
- board text removed: "D"
