File: pcb/revA.sch (KiCad schematic (older format))
At the start: 44 parts, among them P1 USB_OTG, P2 EXP, P3 espprog, P4 BAT, P5 SAMD-PROG, P6 SPI-EXPANSION, SW1 SPST, U1 AP2112K-3.3, U2 SAMD20G18A-M, U3 MCP73831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

Commit message: Updated PCB to the version shipping to kickstarter backers :+1:
Parts:
- P3: footprint user:espprog -> Pin_Headers:Pin_Header_Straight_1x04_Pitch2.54mm
Changed lines of the file:
@@
 F 0 "P3" H 8550 1025 50  0000 C CNN
 F 1 "espprog" V 8650 775 50  0000 C CNN
-F 2 "user:espprog" H 8550 775 50  0001 C CNN
+F 2 "Pin_Headers:Pin_Header_Straight_1x04_Pitch2.54mm" H 8550 775 50  0001 C CNN
 F 3 "" H 8550 775 50  0000 C CNN
 	1    8550 775
